File: Hardware/mb/mb.kicad_pcb (KiCad board)
At the start: 4 copper layers, 93.5 x 69.5 mm, 102 parts, among them J10 PJ-014CH-SMT-TR, J2 Micro_SD_Card_Det_Hirose_DM3AT, J3 B2B-XH-A, J4 USB4105GFA, J5 FFC2B28-12-G, J6 B2B-XH-A, J7 FFC2B28-10-G, J8 F32Q-1A7H1-11030, J9 6871XX149022_687106149022, Q1 2N7002, U1 BQ25895RTWR, U2 RT9742GGJ5, U3 STM6601, U4 TPD2EUSB30, U5 SC0671, U6 TPS61169DCKR

Commit message: .
Routing:
- net GND: vias 301 -> 302
Other:
- board text removed: "2040"
- board text removed: "5v"
- board text removed: "Batt"
- board text removed: "By suya10933"
- board text removed: "CM4 lite"
- board text removed: "DC 12v"
- board text removed: "Ground"
- board text removed: "Lcd"
- board text removed: "Power Btn"
- board text removed: "Rtck"
- board text removed: "SD Card"
- board text removed: "SHH mb v0"
- board text removed: "TLV320"
- board text removed: "Tck"
- board text removed: "Tdi"
- board text removed: "Tdo"
- board text removed: "Tms"
- board text removed: "Touch Pad"
- board text removed: "Trst"
- board text removed: "USB C"
- board text removed: "Uart Rx"
- board text removed: "Uart Tx"
