File: Hardware/mb_v2/mb_v2.kicad_pcb (KiCad board)
At the start: 4 copper layers, 72 x 69.5 mm, 118 parts, among them J1 USB4105GFA, J11 22035025, J2 FFC2B28-22-G_REVA, J3 Micro_SD_Card_Det_Hirose_DM3AT, J4 6871XX149022_687106149022, J5 F32Q-1A7H1-11030, J6 FFC2B28-22-G_REVA, Q2 Q_PMOS_GSD, Q3 Q_NMOS_GSD, Q4 2N7002, Q5 2N7002, Q6 2N7002, U1 MAX77751CEFG_, U10 RP2354A, U2 SC0671, U3 TPS22965DSGR, U4 RT9742GGJ5, U7 TLV75733PDBV, U8 TPD4EUSB30, U9 TPS61169DCKR, Y1 Crystal

Commit message: shh
Routing:
- net +3V3: track 51.3 -> 52.6 mm
- net GND: vias 442 -> 441

Commit message: .
Parts:
- J2, J6, R27, R30: moved to B.Cu
- turned J2 to 90 degrees
- turned J6 to 90 degrees
Connections:
- J2 pad 1: GND -> +5V
- J2 pad 10: GND -> /BTN_CP
- J2 pad 11: /JS_ADC_SDA -> /JS_ADC_SCL
- J2 pad 12: /JS_ADC_SCL -> /JS_ADC_SDA
- J2 pad 13: /BTN_CP -> GND
- J2 pad 14: /BTN_~{PL} -> /TLV320_SDA
- J2 pad 15: /BTN_~{Q7} -> /TLV320_SCL
- J2 pad 17: +3V3_CTRL -> /TLV320_DIN
- J2 pad 18: +3V3_CTRL -> /TLV320_WCLK
- J2 pad 19: GND -> /TLV320_DOUT
- J2 pad 2: /TLV320_BCLK -> +5V
- J2 pad 20: +5V -> /AUDIO_~{RESET}
- J2 pad 21: +5V -> /TLV320_BCLK
- J2 pad 22: +5V -> GND
- J2 pad 3: /AUDIO_~{RESET} -> +5V
- J2 pad 4: /TLV320_DOUT -> GND
- J2 pad 5: /TLV320_WCLK -> +3V3_CTRL
- J2 pad 6: /TLV320_DIN -> +3V3_CTRL
- J2 pad 8: /TLV320_SCL -> /BTN_~{Q7}
- J2 pad 9: /TLV320_SDA -> /BTN_~{PL}
- J6 pad 1: /RUN_PG -> unconnected-(J6-Pad1)
- J6 pad 10: /ARM_TRST -> GND
- J6 pad 11: /ARM_TCK -> /ARM_TDI
- J6 pad 12: /ARM_TDI -> /ARM_TCK
- J6 pad 13: GND -> /ARM_TRST
- J6 pad 14: /SWDIO -> /ARM_TDO
- J6 pad 15: /SWCLK -> /ARM_TMS
- J6 pad 16: GND -> /ARM_RTCK
- J6 pad 17: /2354_UART_TX -> GND
- J6 pad 18: /2354_UART_RX -> /UART_RX
- J6 pad 19: unconnected-(J6-Pad19) -> /UART_TX
- J6 pad 2: /~{RPIBOOT} -> unconnected-(J6-Pad2)
- J6 pad 20: unconnected-(J6-Pad20) -> /GLOBAL_EN
- J6 pad 21: unconnected-(J6-Pad21) -> /~{RPIBOOT}
- J6 pad 22: unconnected-(J6-Pad22) -> /RUN_PG
- J6 pad 3: /GLOBAL_EN -> unconnected-(J6-Pad3)
- J6 pad 4: /UART_TX -> unconnected-(J6-Pad4)
- J6 pad 5: /UART_RX -> /2354_UART_RX
- J6 pad 6: GND -> /2354_UART_TX
- J6 pad 7: /ARM_RTCK -> GND
- J6 pad 8: /ARM_TMS -> /SWCLK
- J6 pad 9: /ARM_TDO -> /SWDIO
Routing:
- net +3V3_CTRL: track 255.9 -> 251.5 mm, vias 11 -> 10
- net /GLOBAL_EN: track 120.1 -> 123.6 mm, vias 4 -> 2
- net /TLV320_BCLK: track 55.6 -> 54.4 mm, vias 2 -> 3
- net /TLV320_SDA: track 59.8 -> 58.6 mm, vias 2 -> 3
- net /TLV320_WCLK: track 54.5 -> 53.3 mm, vias 0 -> 1
- net /TLV320_SCL: track 57.0 -> 55.8 mm, vias 2 -> 3
- net /AUDIO_~{RESET}: track 52.2 -> 51.0 mm, vias 0 -> 1
- net /TLV320_DIN: track 57.3 -> 56.1 mm, vias 2 -> 3
- net /TLV320_DOUT: track 56.9 -> 55.7 mm, vias 2 -> 3
- net +5V: track 193.3 -> 192.2 mm, vias 19 -> 18
- net /ARM_TDI: track 41.8 -> 41.0 mm, vias 2 -> 1
- net /SWCLK: track 73.1 -> 72.4 mm, vias 4 -> 3
- net /SWDIO: track 74.9 -> 74.3 mm, vias 4 -> 3
- net /2354_UART_RX: track 69.3 -> 68.7 mm, vias 2 -> 1
- net /ARM_TCK: track 42.5 -> 41.9 mm, vias 2 -> 1
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Other:
- board text added: "suya@tuta.com / suya10933.neocities.org"
- board text removed: "suya@tuta.com"

Commit message: mb_v2 update
Parts:
- removed C1, C10, C9: 2u2, Capacitor_SMD:C_0805_2012Metric
- removed C7, C8: 10u, Capacitor_SMD:C_0805_2012Metric
- removed D1: HSMG-C110, HSMG-C110:LED_HSMG-C110
- removed J11: 22035025, 22035025:CONN_22035025_MOL
- removed J4: 6871XX149022_687106149022, 6871XX149022_687106149022:687106149022
- removed R1, R2: 20k, Resistor_SMD:R_0603_1608Metric
- removed R3: 20k5~6k65, Resistor_SMD:R_0603_1608Metric
- removed R4: 8k06, Resistor_SMD:R_0603_1608Metric
- removed R5: 1k, Resistor_SMD:R_0603_1608Metric
- removed TP2: VSYS, TestPoint:TestPoint_Pad_1.0x1.0mm
- removed U1: MAX77751CEFG_, MAX77751CEFG_:IC_MAX77751CEFG_
- added C54: 1u, Capacitor_SMD:C_0805_2012Metric, F.Cu at (70.2, 108.9)
- added C55: 10u, Capacitor_SMD:C_0805_2012Metric, F.Cu at (77.6, 108.3)
- added C58: 100n, Capacitor_SMD:C_0805_2012Metric, F.Cu at (74.1, 108.3)
- added C59: 10u, Capacitor_SMD:C_0805_2012Metric, F.Cu at (74.9, 115.6)
- added D7: 1N4148W, Diode_SMD:D_SOD-123, F.Cu at (98.9, 99.0)
- added J7: 22057025, 22057025:CONN_22057025_MOL, F.Cu at (109.9, 112.1)
- added J9: F3311A7H121030E200, F3311A7H121030E200:AMPHENOL_F3311A7H121030E200, B.Cu at (96.0, 84.5)
- added R12: 900k, Resistor_SMD:R_0603_1608Metric, F.Cu at (66.7, 109.8)
- added R16: 5k6, Resistor_SMD:R_0603_1608Metric, F.Cu at (71.0, 111.9)
- added R17: 5k23, Resistor_SMD:R_0603_1608Metric, F.Cu at (68.9, 115.4)
- added R37: 7k5, Resistor_SMD:R_0603_1608Metric, F.Cu at (67.4, 115.4)
- added R38: 10k, Resistor_SMD:R_0603_1608Metric, F.Cu at (109.4, 91.1)
- added R39: 200k, Resistor_SMD:R_0603_1608Metric, F.Cu at (107.8, 91.1)
- added R40: 2k2, Resistor_SMD:R_0603_1608Metric, B.Cu at (56.5, 70.5)
- added R41: 2k2, Resistor_SMD:R_0603_1608Metric, B.Cu at (56.5, 72.0)
- added U5: TUSB320, Package_DFN_QFN:Texas_X2QFN-12_1.6x1.6mm_P0.4mm, F.Cu at (66.7, 107.6)
- added U6: BQ25628ERYKR, footprints:WQFN-HR18__RYK_TEX, F.Cu at (74.0, 111.6)
- C4: value 22u -> 47n
- C5: value 10u -> 4u7
- C6: footprint Capacitor_SMD:C_0603_1608Metric -> Capacitor_SMD:C_0805_2012Metric
- J5: value F32Q-1A7H1-11030 -> 5034800600; footprint F32Q-1A7H1-11030:AMPHENOL_F32Q-1A7H1-11030 -> 5034800600:503480-0600_MOL
- L1: value DFE252010F-R47M=P2 -> SPM3020T-1R0M-LR; footprint DFE252010F-R47M_P2:INDC2520X100N -> SPM3020T-1R0M-LR:IND_SPM3020T-1R0M-LR
- moved J5 23.0 mm to (116.0, 68.5), turned to 90 degrees
- moved C5 6.98 mm to (69.2, 111.7), turned to -90 degrees
- moved C6 5.37 mm to (64.1, 107.6), turned to -90 degrees
- moved C4 4.65 mm to (70.2, 106.9), turned to 0 degrees
- moved L1 4.04 mm to (78.2, 111.6), turned to -90 degrees
- moved C35 2.80 mm to (77.0, 115.6), turned to -90 degrees
- moved C36 2.25 mm to (79.1, 115.6), turned to -90 degrees
- moved C2 0.81 mm to (72.8, 115.6)
- moved C3 0.80 mm to (70.7, 115.6)
- moved D3 0.54 mm to (108.0, 52.5)
- moved S1 0.50 mm to (100.5, 52.5)
- moved R7 0.40 mm to (113.0, 52.8)
- moved R24 0.30 mm to (111.5, 52.8)
- moved U4 0.30 mm to (115.5, 52.8)
Connections:
- C4 pad 1: Net-(U1-BYP) -> Net-(U6-BTST)
- C4 pad 2: GND -> Net-(U6-SW)
- C5 pad 1: Net-(U1-BYP) -> Net-(U6-REGN)
- C6 pad 1: Net-(U1-BST) -> +3V3_CTRL
- C6 pad 2: Net-(U1-LX) -> GND
- J5 pad 1: /ER-TFT050-10_LEDK -> +3V3_CTRL
- J5 pad 2: /ER-TFT050-10_LEDK -> /TP_INT
- J5 pad 3: /ER-TFT050-10_LEDK -> /TP_RST
- J5 pad 4: /ER-TFT050-10_LEDA -> /PMIC_I2C_SDA
- J5 pad 5: /ER-TFT050-10_LEDA -> /PMIC_I2C_SCL
- J5 pad 6: /ER-TFT050-10_LEDA -> GND
- J5 pad 7: GND -> (no net)
- J5 pad 8: GND -> (no net)
- L1 pad 1: Net-(U1-LX) -> Net-(U6-SW)
- R35 pad 1: /TP_SDA -> /PMIC_I2C_SDA
- R36 pad 1: /TP_SCL -> /PMIC_I2C_SCL
- U10 pad 27: unconnected-(U10-GPIO16-Pad27) -> /BQ25628_~{INT}
- U10 pad 28: unconnected-(U10-GPIO17-Pad28) -> /TUSB320_~{INT}
- U10 pad 40: /TP_SDA -> /PMIC_I2C_SDA
- U10 pad 41: /TP_SCL -> /PMIC_I2C_SCL
Routing:
- net /PMIC_I2C_SDA: track 0.00 -> 94.9 mm, vias 0 -> 6
- net /PMIC_I2C_SCL: track 0.00 -> 94.4 mm, vias 0 -> 6
- net /TUSB320_~{INT}: track 0.00 -> 70.4 mm, vias 0 -> 5
- net /BQ25628_~{INT}: track 0.00 -> 63.7 mm, vias 0 -> 5
- net +3V3: track 52.6 -> 101.9 mm
- net VSYS: track 170.9 -> 133.9 mm, vias 7 -> 4
- net VBUS: track 26.6 -> 60.0 mm, vias 3 -> 17
- net /TLV320_SDA: track 58.6 -> 78.2 mm, vias 3 -> 5
- net /MAX77751_STAT: track 16.7 -> 0.00 mm, vias 2 -> 0
- net /TLV320_SCL: track 55.8 -> 70.2 mm, vias 3 -> 5
- net /TP_SDA: track 13.9 -> 0.00 mm, vias 2 -> 0
- net /TP_SCL: track 13.8 -> 0.00 mm, vias 2 -> 0
- net Net-(U1-LX): track 13.0 -> 0.00 mm
- net /USBC_CC2: track 26.1 -> 13.5 mm, vias 2 -> 0
- net +BATT: track 87.9 -> 100.4 mm
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- added copper zone on B.Cu, net Net-(U6-SW)
- added copper zone on F.Cu, net Net-(U6-SW)
- added copper zone on B.Cu, net VBUS
- added copper zone on F.Cu, net VBUS
Other:
- outline, holes or cut-outs redrawn
