File: Hardware/mb_v2/mb_v2.kicad_sch (KiCad schematic)
At the start: 118 parts, among them J1 USB4105GFA, J11 22035025, J2 FFC2B28-22-G_REVA, J3 Micro_SD_Card_Det_Hirose_DM3AT, J4 6871XX149022_687106149022, J5 F32Q-1A7H1-11030, J6 FFC2B28-22-G_REVA, Q2 Q_PMOS_GSD, Q3 Q_NMOS_GSD, Q4 2N7002, Q5 2N7002, Q6 2N7002, U1 MAX77751CEFG_, U10 RP2354A, U2 SC0671, U3 TPS22965DSGR, U4 RT9742GGJ5, U7 TLV75733PDBV, U8 TPD4EUSB30, U9 TPS61169DCKR, Y1 Crystal

Commit message: .
Connections:
- net +3V3_CTRL: now also J2.5, J2.6; no longer J2.17, J2.18
- net +5V: now also J2.1, J2.2, J2.3; no longer J2.20, J2.21, J2.22
- net 2354_UART_RX: now also J6.5; no longer J6.18
- net 2354_UART_TX: now also J6.6; no longer J6.17
- net ARM_RTCK: now also J6.16; no longer J6.7
- net ARM_TCK: now also J6.12; no longer J6.11
- net ARM_TDI: now also J6.11; no longer J6.12
- net ARM_TDO: now also J6.14; no longer J6.9
- net ARM_TMS: now also J6.15; no longer J6.8
- net ARM_TRST: now also J6.13; no longer J6.10
- net AUDIO_~{RESET}: now also J2.20; no longer J2.3
- net BTN_CP: now also J2.10; no longer J2.13
- net BTN_~{PL}: now also J2.9; no longer J2.14
- net BTN_~{Q7}: now also J2.8; no longer J2.15
- net GLOBAL_EN: now also J6.20; no longer J6.3
- net GND: now also J2.13, J2.22, J2.4, J6.10, J6.17, J6.7; no longer J2.1, J2.10, J2.19, J6.13, J6.16, J6.6
- net JS_ADC_SCL: now also J2.11; no longer J2.12
- net JS_ADC_SDA: now also J2.12; no longer J2.11
- net RUN_PG: now also J6.22; no longer J6.1
- net SWCLK: now also J6.8; no longer J6.15
- net SWDIO: now also J6.9; no longer J6.14
- net TLV320_BCLK: now also J2.21; no longer J2.2
- net TLV320_DIN: now also J2.17; no longer J2.6
- net TLV320_DOUT: now also J2.19; no longer J2.4
- net TLV320_SCL: now also J2.15; no longer J2.8
- net TLV320_SDA: now also J2.14; no longer J2.9
- net TLV320_WCLK: now also J2.18; no longer J2.5
- net UART_RX: now also J6.18; no longer J6.5
- net UART_TX: now also J6.19; no longer J6.4
- net ~{RPIBOOT}: now also J6.21; no longer J6.2

Commit message: mb_v2 update
Parts:
- removed C1, C10, C9: 2u2, Capacitor_SMD:C_0805_2012Metric, symbol Device:C
- removed C7, C8: 10u, Capacitor_SMD:C_0805_2012Metric, symbol Device:C
- removed D1: HSMG-C110, HSMG-C110:LED_HSMG-C110, symbol HSMG-C110:HSMG-C110
- removed J11: 22035025, 22035025:CONN_22035025_MOL, symbol 22035025:22035025
- removed J4: 6871XX149022_687106149022, 6871XX149022_687106149022:687106149022, symbol 6871XX149022_687106149022:6871XX149022_687106149022
- removed J5: F32Q-1A7H1-11030, F32Q-1A7H1-11030:AMPHENOL_F32Q-1A7H1-11030, symbol F32Q-1A7H1-11030:F32Q-1A7H1-11030
- removed L1: DFE252010F-R47M=P2, DFE252010F-R47M_P2:INDC2520X100N, symbol DFE252010F-R47M_P2:DFE252010F-R47M=P2
- removed R1, R2: 20k, Resistor_SMD:R_0603_1608Metric, symbol Device:R
- removed R3: 20k5~6k65, Resistor_SMD:R_0603_1608Metric, symbol Device:R
- removed R4: 8k06, Resistor_SMD:R_0603_1608Metric, symbol Device:R
- removed R5: 1k, Resistor_SMD:R_0603_1608Metric, symbol Device:R
- removed TP2: VSYS, TestPoint:TestPoint_Pad_1.0x1.0mm, symbol Connector:TestPoint
- removed U1: MAX77751CEFG_, MAX77751CEFG_:IC_MAX77751CEFG_, symbol MAX77751CEFG_:MAX77751CEFG_
- added C54: 1u, Capacitor_SMD:C_0805_2012Metric, symbol Device:C
- added C55, C59: 10u, Capacitor_SMD:C_0805_2012Metric, symbol Device:C
- added C58: 100n, Capacitor_SMD:C_0805_2012Metric, symbol Device:C
- added D7: 1N4148W, Diode_SMD:D_SOD-123, symbol Diode:1N4148W
- added J5: 5034800600, 5034800600:503480-0600_MOL, symbol 5034800600:5034800600
- added J7: 22057025, 22057025:CONN_22057025_MOL, symbol 22057025:22057025
- added J9: F3311A7H121030E200, F3311A7H121030E200:AMPHENOL_F3311A7H121030E200, symbol F3311A7H121030E200:F3311A7H121030E200
- added L1: SPM3020T-1R0M-LR, SPM3020T-1R0M-LR:IND_SPM3020T-1R0M-LR, symbol SPM3020T-1R0M-LR:SPM3020T-1R0M-LR
- added R12: 900k, Resistor_SMD:R_0603_1608Metric, symbol Device:R
- added R16: 5k6, Resistor_SMD:R_0603_1608Metric, symbol Device:R
- added R17: 5k23, Resistor_SMD:R_0603_1608Metric, symbol Device:R
- added R37: 7k5, Resistor_SMD:R_0603_1608Metric, symbol Device:R
- added R38: 10k, Resistor_SMD:R_0603_1608Metric, symbol Device:R
- added R39: 200k, Resistor_SMD:R_0603_1608Metric, symbol Device:R
- added R40, R41: 2k2, Resistor_SMD:R_0603_1608Metric, symbol Device:R
- added U5: TUSB320, Package_DFN_QFN:Texas_X2QFN-12_1.6x1.6mm_P0.4mm, symbol Interface_USB:TUSB320
- added U6: BQ25628ERYKR, footprints:WQFN-HR18__RYK_TEX, symbol 2026-08-12_05-02-26:BQ25628ERYKR
- C4: value 22u -> 47n
- C5: value 10u -> 4u7
- C6: footprint Capacitor_SMD:C_0603_1608Metric -> Capacitor_SMD:C_0805_2012Metric
Connections:
- net +3V3: now also R40.2, R41.2
- net +3V3_CTRL: now also C6.1, J5.1, J9.3, J9.5, J9.6, R38.2, R39.2, U5.12 (VDD)
- net +BATT: now also J7.1, U6.8 (BAT)
- net ER-TFT050-10_CLKN: now also J9.16
- net ER-TFT050-10_CLKP: now also J9.15
- net ER-TFT050-10_D0N: now also J9.10
- net ER-TFT050-10_D0P: now also J9.9
- net ER-TFT050-10_D1N: now also J9.13
- net ER-TFT050-10_D1P: now also J9.12
- net ER-TFT050-10_LEDA: now also J9.25, J9.26, J9.27
- net ER-TFT050-10_LEDK: now also J9.28, J9.29, J9.30
- net ER-TFT050-10_RST: now also J9.2
- net GND: now also C6.2, C54.2, C55.2, C58.2, C59.2, J5.6, J7.2, J9.1, J9.11, J9.14, J9.17, J9.20, J9.23, J9.24, J9.4, J9.7, J9.8, R16.2, R37.2, U5.10 (GND), U5.11 (~{EN}), U5.3 (PORT), U5.5 (ADDR), U6.14 (*CE), U6.15 (GND); no longer C4.2
- net TLV320_SCL: now also R40.1
- net TLV320_SDA: now also R41.1
- net TP_INT: now also J5.2
- net TP_RST: now also J5.3
- net USBC_CC1: now also U5.1 (CC1)
- net USBC_CC2: now also U5.2 (CC2)
- net VBUS: now also C54.1, D7.2 (A), R12.1, U6.18 (VBUS)
- net VSYS: now also C59.1, L1.2, U6.9 (SYS)
- net at D4.1 (K), D6.1 (K), R33.1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: now also D7.1 (K)
- net BQ25628_~{INT}: now reaches U10.27 (GPIO16)
- net BQ25628_~{INT}: now also R38.1, U6.11 (*INT)
- net TUSB320_~{INT}: now reaches U10.28 (GPIO17)
- net TUSB320_~{INT}: now also R39.1, U5.6 (~{INT}/OUT3)
- net at C5.1: now also U6.2 (REGN); no longer C4.1
- net TP_SCL renamed PMIC_I2C_SCL
- net PMIC_I2C_SCL: now also J5.5, U5.8 (SCL/OUT2), U6.13 (SCL)
- net TP_SDA renamed PMIC_I2C_SDA
- net PMIC_I2C_SDA: now also J5.4, U5.7 (SDA/OUT1), U6.12 (SDA)
- new net: C4.2, L1.1, U6.16 (SW)
- new net: C55.1, C58.1, U6.17 (PMID)
- new net: C4.1, U6.1 (BTST)
- new net: R16.1, U6.4 (ILIM)
- new net: R17.1, U6.5 (TS_BIAS)
- new net: R17.2, R37.1, U6.6 (TS)
- new net: R12.2, U5.4 (VBUS_DET)
- no-connect marks 117 -> 121
Other:
- moved on the sheet: Q5, R31, R32
